File: hertzschlag/hertzschlag.kicad_sch (KiCad schematic)
At the start: 28 parts, among them IC1 TB67H450FNG,EL, IC2 TB67H450FNG,EL, J1 TB_1X2, J12 Conn_01x04_Female, J14 Conn_01x03_Male, J17 Conn_01x30_Pin, J2 Conn_01x03_Male, J4 MotorA, J5 MotorB, SW1 SW_Push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

Commit message: Changes on PCB.
Changes to Footprints, Routing, Alignment.
And no more falling alita on the front Silk screen (sad).
Parts:
- removed C1: 22uf, Capacitor_SMD:C_0805_2012Metric_Pad1.18x1.45mm_HandSolder, symbol Device:C
- C3, C5: footprint Capacitor_Tantalum_SMD:CP_EIA-3216-18_Kemet-A_HandSolder -> Capacitor_Tantalum_SMD:CP_EIA-6032-15_Kemet-U_HandSolder
- renumbered J4 to J2, J5 to J3, J17 to J4, J12 to J5, J2 to J6, J14 to J7
Changed lines of the file:
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@@
 	)
 	(junction
-		(at 81.28 39.37)
-		(diameter 0)
-		(color 0 0 0 0)
-	)
-	(junction
 		(at 157.48 43.18)
 		(diameter 0)
@@
 	)
 	(junction
-		(at 87.63 31.75)
-		(diameter 0)
-		(color 0 0 0 0)
-	)
-	(junction
 		(at 128.27 81.28)
 		(diameter 0)
@@
 	(wire
 		(pts
-			(xy 78.74 31.75) (xy 87.63 31.75)
+			(xy 78.74 31.75) (xy 93.98 31.75)
 		)
 		(stroke
@@
 	(wire
 		(pts
-			(xy 81.28 39.37) (xy 87.63 39.37)
-		)
-		(stroke
-			(width 0)
-			(type default)
-		)
-	)
-	(wire
-		(pts
 			(xy 157.48 27.94) (xy 157.48 31.75)
 		)
@@
 		)
 	)
-	(wire
-		(pts
-			(xy 87.63 31.75) (xy 93.98 31.75)
-		)
-		(stroke
-			(width 0)
-			(type default)
-		)
-	)
 	(polyline
 		(pts
@@
 	(wire
 		(pts
-			(xy 81.28 44.45) (xy 81.28 39.37)
-		)
-		(stroke
-			(width 0)
-			(type default)
-		)
-	)
-	(wire
-		(pts
 			(xy 157.48 43.18) (xy 162.56 43.18)
 		)
@@
 	(wire
 		(pts
-			(xy 81.28 39.37) (xy 81.28 35.56)
+			(xy 81.28 35.56) (xy 81.28 44.45)
 		)
 		(stroke
@@
 			)
 		)
-		(property "Footprint" "Capacitor_Tantalum_SMD:CP_EIA-3216-18_Kemet-A_HandSolder"
+		(property "Footprint" "Capacitor_Tantalum_SMD:CP_EIA-6032-15_Kemet-U_HandSolder"
 			(at 129.2352 88.9 0)
 			(effects
@@
 			)
 		)
-		(property "Footprint" "Capacitor_Tantalum_SMD:CP_EIA-3216-18_Kemet-A_HandSolder"
+		(property "Footprint" "Capacitor_Tantalum_SMD:CP_EIA-6032-15_Kemet-U_HandSolder"
 			(at 129.2352 128.27 0)
 			(effects
@@
 		(on_board yes)
 		(dnp no)
-		(property "Reference" "J17"
+		(property "Reference" "J4"
 			(at 30.48 151.384 0)
 			(effects
@@
 			(project ""
 				(path "/f154c6d1-45a5-4a23-92c8-ac7beedeed65"
-					(reference "J17")
+					(reference "J4")
 					(unit 1)
 				)
@@
 		(dnp no)
 		(fields_autoplaced yes)
-		(property "Reference" "J5"
+		(property "Reference" "J3"
 			(at 193.04 135.8899 0)
 			(effects
@@
 			(project "MiniSumo_Nano"
 				(path "/f154c6d1-45a5-4a23-92c8-ac7beedeed65"
-					(reference "J5")
+					(reference "J3")
 					(unit 1)
 				)
@@
 		(dnp no)
 		(fields_autoplaced yes)
-		(property "Reference" "J2"
+		(property "Reference" "J6"
 			(at 63.5 115.5699 0)
 			(effects
@@
 			(project "MiniSumo_Nano"
 				(path "/f154c6d1-45a5-4a23-92c8-ac7beedeed65"
-					(reference "J2")
+					(reference "J6")
 					(unit 1)
 				)
@@
 		(on_board yes)
 		(dnp no)
-		(property "Reference" "J12"
+		(property "Reference" "J5"
 			(at 58.166 98.044 0)
 			(effects
@@
 			(project "MiniSumo_Nano"
 				(path "/f154c6d1-45a5-4a23-92c8-ac7beedeed65"
-					(reference "J12")
+					(reference "J5")
 					(unit 1)
 				)
@@
 		(on_board yes)
 		(dnp no)
-		(property "Reference" "J14"
+		(property "Reference" "J7"
 			(at 63.5 132.0799 0)
 			(effects
@@
 			(project "MiniSumo_Nano"
 				(path "/f154c6d1-45a5-4a23-92c8-ac7beedeed65"
-					(reference "J14")
+					(reference "J7")
 					(unit 1)
 				)
@@
 		(dnp no)
 		(fields_autoplaced yes)
-		(property "Reference" "J4"
+		(property "Reference" "J2"
 			(at 191.77 97.7899 0)
 			(effects
@@
 			(project "MiniSumo_Nano"
 				(path "/f154c6d1-45a5-4a23-92c8-ac7beedeed65"
-					(reference "J4")
+					(reference "J2")
 					(unit 1)
 				)
@@
 					(unit 1)
 				)
-			)
-		)
-	)
-	(symbol
-		(lib_id "Device:C")
-		(at 87.63 35.56 0)
-		(unit 1)
-		(exclude_from_sim no)
-		(in_bom yes)
-		(on_board yes)
-		(dnp no)
-		(fields_autoplaced yes)
-		(property "Reference" "C1"
-			(at 91.44 34.2899 0)
-			(effects
-				(font
-					(size 1.27 1.27)
-				)
-				(justify left)
-			)
-		)
-		(property "Value" "22uf"
-			(at 91.44 36.8299 0)
-			(effects
-				(font
-					(size 1.27 1.27)
-				)
-				(justify left)
-			)
-		)
-		(property "Footprint" "Capacitor_SMD:C_0805_2012Metric_Pad1.18x1.45mm_HandSolder"
-			(at 88.5952 39.37 0)
-			(effects
-				(font
-					(size 1.27 1.27)
-				)
-				(hide yes)
-			)
-		)
-		(property "Datasheet" "~"
-			(at 87.63 35.56 0)
-			(effects
-				(font
-					(size 1.27 1.27)
-				)
-				(hide yes)
-			)
-		)
-		(property "Description" "Unpolarized capacitor"
-			(at 87.63 35.56 0)
-			(effects
-				(font
-					(size 1.27 1.27)
-				)
-				(hide yes)
-			)
-		)
-		(pin "1"
-		)
-		(pin "2"
-		)
-		(instances
-			(project "MiniSumo_Nano"
-				(path "/f154c6d1-45a5-4a23-92c8-ac7beedeed65"
-					(reference "C1")
-					(unit 1)
-				)
