File: hertzschlag/hertzschlag.kicad_pcb (KiCad board)
At the start: 4 copper layers, 85.5 x 28 mm, 32 parts, among them IC1 TB67H450FNG,EL, IC2 TB67H450FNG,EL, J1 TB_1X2, J2 MotorA, J3 MotorB, J4 Conn_01x30_Pin, J8 Extra, SW1 SW_Push, SW2 SW_Push, SW3 SW_Push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

Commit message: PCB
Other:
- copper layers 4 -> 2
Changed lines of the file:
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@@
 	(layers
 		(0 "F.Cu" signal)
-		(4 "In1.Cu" signal)
-		(6 "In2.Cu" signal)
 		(2 "B.Cu" signal)
 		(9 "F.Adhes" user "F.Adhesive")
@@
 			)
 			(layer "dielectric 1"
-				(type "prepreg")
-				(thickness 0.1)
-				(material "FR4")
-				(epsilon_r 4.5)
-				(loss_tangent 0.02)
-			)
-			(layer "In1.Cu"
-				(type "copper")
-				(thickness 0.035)
-			)
-			(layer "dielectric 2"
 				(type "core")
-				(thickness 1.24)
-				(material "FR4")
-				(epsilon_r 4.5)
-				(loss_tangent 0.02)
-			)
-			(layer "In2.Cu"
-				(type "copper")
-				(thickness 0.035)
-			)
-			(layer "dielectric 3"
-				(type "prepreg")
-				(thickness 0.1)
+				(thickness 1.51)
 				(material "FR4")
 				(epsilon_r 4.5)
@@
 	)
 	(segment
-		(start 161.05 109.3)
-		(end 162.36 107.99)
+		(start 146 108.14)
+		(end 147.14 109.28)
 		(width 1.5)
 		(layer "F.Cu")
@@
 	)
 	(segment
-		(start 146 108.14)
-		(end 147.14 109.28)
-		(width 1.5)
-		(layer "F.Cu")
-		(net 8)
-	)
-	(segment
 		(start 111.45625 99.81875)
 		(end 112.18825 99.81875)
@@
 	)
 	(segment
-		(start 157.04 109.3)
-		(end 161.05 109.3)
-		(width 1.5)
-		(layer "F.Cu")
-		(net 8)
-	)
-	(segment
-		(start 147.14 109.28)
-		(end 157.02 109.28)
-		(width 1.5)
-		(layer "F.Cu")
-		(net 8)
-	)
-	(segment
 		(start 157.02 109.28)
 		(end 157.04 109.3)
@@
 	)
 	(segment
+		(start 147.14 109.28)
+		(end 157.02 109.28)
+		(width 1.5)
+		(layer "F.Cu")
+		(net 8)
+	)
+	(segment
 		(start 122.195 99.375)
 		(end 122.195 98.454)
@@
 		(layer "F.Cu")
 		(net 8)
+	)
+	(segment
+		(start 157.04 109.3)
+		(end 161.05 109.3)
+		(width 1.5)
+		(layer "F.Cu")
+		(net 8)
+	)
+	(segment
+		(start 161.05 109.3)
+		(end 162.36 107.99)
+		(width 1.5)
+		(layer "F.Cu")
+		(net 8)
